File: src/CC3200.kicad_pcb (KiCad board)
At the start: 2 copper layers, 0 parts

Commit message: Footprint and Symbol updated
Parts:
- added U1: CC3200, CC3200, F.Cu at (213.4, 148.6)
Other:
- board outline added: 25.4 x 21.6 mm
Changed lines of the file:
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@@
     (area 0 0 0 0)
     (thickness 1.6)
-    (drawings 0)
+    (drawings 4)
     (tracks 0)
     (zones 0)
-    (modules 0)
+    (modules 1)
     (nets 1)
   )
@@
     (pad_to_mask_clearance 0)
     (aux_axis_origin 0 0)
-    (visible_elements FFFFFFBF)
+    (visible_elements 7FFFFFFF)
     (pcbplotparams
       (layerselection 3178497)
@@
     (add_net "")
   )
+  (module CC3200 (layer F.Cu)
+    (at 213.36 148.59)
+    (fp_text reference U1 (at 0 -6.5) (layer F.SilkS)
+      (effects (font (size 1 1) (thickness 0.15)))
+    )
+    (fp_text value CC3200 (at 0 6.48) (layer F.SilkS)
+      (effects (font (size 1 1) (thickness 0.15)))
+    )
+    (fp_text user 1 (at -4.4 5.14) (layer F.SilkS)
+      (effects (font (size 0.5 0.5) (thickness 0.125)))
+    )
+    (fp_circle (center -3.72 3.72) (end -3.52 3.73) (layer F.SilkS) (width 0.15))
+    (fp_line (start -4.575 4.575) (end -4.575 -4.575) (layer F.SilkS) (width 0.15))
+    (fp_line (start -4.575 -4.575) (end 4.575 -4.575) (layer F.SilkS) (width 0.15))
+    (fp_line (start 4.575 -4.575) (end 4.575 4.575) (layer F.SilkS) (width 0.15))
+    (fp_line (start 4.575 4.575) (end -4.575 4.575) (layer F.SilkS) (width 0.15))
+    (pad 57 smd oval (at -4.75 0.25 90) (size 0.3 1.5)
+      (layers F.Cu F.Paste F.Mask)
+    )
+    (pad 58 smd oval (at -4.75 0.75 90) (size 0.3 1.5)
+      (layers F.Cu F.Paste F.Mask)
+    )
+    (pad 60 smd oval (at -4.75 1.75 90) (size 0.3 1.5)
+      (layers F.Cu F.Paste F.Mask)
+    )
+    (pad 59 smd oval (at -4.75 1.25 90) (size 0.3 1.5)
+      (layers F.Cu F.Paste F.Mask)
+    )
+    (pad 63 smd oval (at -4.75 3.25 90) (size 0.3 1.5)
+      (layers F.Cu F.Paste F.Mask)
+    )
+    (pad 64 smd oval (at -4.75 3.75 90) (size 0.3 1.5)
+      (layers F.Cu F.Paste F.Mask)
+    )
+    (pad 62 smd oval (at -4.75 2.75 90) (size 0.3 1.5)
+      (layers F.Cu F.Paste F.Mask)
+    )
+    (pad 61 smd oval (at -4.75 2.25 90) (size 0.3 1.5)
+      (layers F.Cu F.Paste F.Mask)
+    )
+    (pad 53 smd oval (at -4.75 -1.75 90) (size 0.3 1.5)
+      (layers F.Cu F.Paste F.Mask)
+    )
+    (pad 54 smd oval (at -4.75 -1.25 90) (size 0.3 1.5)
+      (layers F.Cu F.Paste F.Mask)
+    )
+    (pad 56 smd oval (at -4.75 -0.25 90) (size 0.3 1.5)
+      (layers F.Cu F.Paste F.Mask)
+    )
+    (pad 55 smd oval (at -4.75 -0.75 90) (size 0.3 1.5)
+      (layers F.Cu F.Paste F.Mask)
+    )
+    (pad 51 smd oval (at -4.75 -2.75 90) (size 0.3 1.5)
+      (layers F.Cu F.Paste F.Mask)
+    )
+    (pad 52 smd oval (at -4.75 -2.25 90) (size 0.3 1.5)
+      (layers F.Cu F.Paste F.Mask)
+    )
+    (pad 50 smd oval (at -4.75 -3.25 90) (size 0.3 1.5)
+      (layers F.Cu F.Paste F.Mask)
+    )
+    (pad 49 smd oval (at -4.75 -3.75 90) (size 0.3 1.5)
+      (layers F.Cu F.Paste F.Mask)
+    )
+    (pad 32 smd oval (at 4.75 -3.75 90) (size 0.3 1.5)
+      (layers F.Cu F.Paste F.Mask)
+    )
+    (pad 31 smd oval (at 4.75 -3.25 90) (size 0.3 1.5)
+      (layers F.Cu F.Paste F.Mask)
+    )
+    (pad 29 smd oval (at 4.75 -2.25 90) (size 0.3 1.5)
+      (layers F.Cu F.Paste F.Mask)
+    )
+    (pad 30 smd oval (at 4.75 -2.75 90) (size 0.3 1.5)
+      (layers F.Cu F.Paste F.Mask)
+    )
+    (pad 26 smd oval (at 4.75 -0.75 90) (size 0.3 1.5)
+      (layers F.Cu F.Paste F.Mask)
+    )
+    (pad 25 smd oval (at 4.75 -0.25 90) (size 0.3 1.5)
+      (layers F.Cu F.Paste F.Mask)
+    )
+    (pad 27 smd oval (at 4.75 -1.25 90) (size 0.3 1.5)
+      (layers F.Cu F.Paste F.Mask)
+    )
+    (pad 28 smd oval (at 4.75 -1.75 90) (size 0.3 1.5)
+      (layers F.Cu F.Paste F.Mask)
+    )
+    (pad 20 smd oval (at 4.75 2.25 90) (size 0.3 1.5)
+      (layers F.Cu F.Paste F.Mask)
+    )
+    (pad 19 smd oval (at 4.75 2.75 90) (size 0.3 1.5)
+      (layers F.Cu F.Paste F.Mask)
+    )
+    (pad 17 smd oval (at 4.75 3.75 90) (size 0.3 1.5)
+      (layers F.Cu F.Paste F.Mask)
+    )
+    (pad 18 smd oval (at 4.75 3.25 90) (size 0.3 1.5)
+      (layers F.Cu F.Paste F.Mask)
+    )
+    (pad 22 smd oval (at 4.75 1.25 90) (size 0.3 1.5)
+      (layers F.Cu F.Paste F.Mask)
+    )
+    (pad 21 smd oval (at 4.75 1.75 90) (size 0.3 1.5)
+      (layers F.Cu F.Paste F.Mask)
+    )
+    (pad 23 smd oval (at 4.75 0.75 90) (size 0.3 1.5)
+      (layers F.Cu F.Paste F.Mask)
+    )
+    (pad 24 smd oval (at 4.75 0.25 90) (size 0.3 1.5)
+      (layers F.Cu F.Paste F.Mask)
+    )
+    (pad 41 smd oval (at -0.25 -4.75) (size 0.3 1.5)
+      (layers F.Cu F.Paste F.Mask)
+    )
+    (pad 42 smd oval (at -0.75 -4.75) (size 0.3 1.5)
+      (layers F.Cu F.Paste F.Mask)
+    )
+    (pad 44 smd oval (at -1.75 -4.75) (size 0.3 1.5)
+      (layers F.Cu F.Paste F.Mask)
+    )
+    (pad 43 smd oval (at -1.25 -4.75) (size 0.3 1.5)
+      (layers F.Cu F.Paste F.Mask)
+    )
+    (pad 47 smd oval (at -3.25 -4.75) (size 0.3 1.5)
+      (layers F.Cu F.Paste F.Mask)
+    )
+    (pad 48 smd oval (at -3.75 -4.75) (size 0.3 1.5)
+      (layers F.Cu F.Paste F.Mask)
+    )
+    (pad 46 smd oval (at -2.75 -4.75) (size 0.3 1.5)
+      (layers F.Cu F.Paste F.Mask)
+    )
+    (pad 45 smd oval (at -2.25 -4.75) (size 0.3 1.5)
+      (layers F.Cu F.Paste F.Mask)
+    )
+    (pad 37 smd oval (at 1.75 -4.75) (size 0.3 1.5)
+      (layers F.Cu F.Paste F.Mask)
+    )
+    (pad 38 smd oval (at 1.25 -4.75) (size 0.3 1.5)
+      (layers F.Cu F.Paste F.Mask)
+    )
+    (pad 40 smd oval (at 0.25 -4.75) (size 0.3 1.5)
+      (layers F.Cu F.Paste F.Mask)
+    )
+    (pad 39 smd oval (at 0.75 -4.75) (size 0.3 1.5)
+      (layers F.Cu F.Paste F.Mask)
+    )
+    (pad 35 smd oval (at 2.75 -4.75) (size 0.3 1.5)
+      (layers F.Cu F.Paste F.Mask)
+    )
+    (pad 36 smd oval (at 2.25 -4.75) (size 0.3 1.5)
+      (layers F.Cu F.Paste F.Mask)
+    )
+    (pad 34 smd oval (at 3.25 -4.75) (size 0.3 1.5)
+      (layers F.Cu F.Paste F.Mask)
+    )
+    (pad 33 smd oval (at 3.75 -4.75) (size 0.3 1.5)
+      (layers F.Cu F.Paste F.Mask)
+    )
+    (pad 16 smd oval (at 3.75 4.75) (size 0.3 1.5)
+      (layers F.Cu F.Paste F.Mask)
+    )
+    (pad 15 smd oval (at 3.25 4.75) (size 0.3 1.5)
+      (layers F.Cu F.Paste F.Mask)
+    )
+    (pad 13 smd oval (at 2.25 4.75) (size 0.3 1.5)
+      (layers F.Cu F.Paste F.Mask)
+    )
+    (pad 14 smd oval (at 2.75 4.75) (size 0.3 1.5)
+      (layers F.Cu F.Paste F.Mask)
+    )
+    (pad 10 smd oval (at 0.75 4.75) (size 0.3 1.5)
+      (layers F.Cu F.Paste F.Mask)
+    )
+    (pad 9 smd oval (at 0.25 4.75) (size 0.3 1.5)
+      (layers F.Cu F.Paste F.Mask)
+    )
+    (pad 11 smd oval (at 1.25 4.75) (size 0.3 1.5)
+      (layers F.Cu F.Paste F.Mask)
+    )
+    (pad 12 smd oval (at 1.75 4.75) (size 0.3 1.5)
+      (layers F.Cu F.Paste F.Mask)
+    )
+    (pad 4 smd oval (at -2.25 4.75) (size 0.3 1.5)
+      (layers F.Cu F.Paste F.Mask)
+    )
+    (pad 3 smd oval (at -2.75 4.75) (size 0.3 1.5)
+      (layers F.Cu F.Paste F.Mask)
+    )
+    (pad 1 smd oval (at -3.75 4.75) (size 0.3 1.5)
+      (layers F.Cu F.Paste F.Mask)
+    )
+    (pad 2 smd oval (at -3.25 4.75) (size 0.3 1.5)
+      (layers F.Cu F.Paste F.Mask)
+    )
+    (pad 6 smd oval (at -1.25 4.75) (size 0.3 1.5)
+      (layers F.Cu F.Paste F.Mask)
+    )
+    (pad 5 smd oval (at -1.75 4.75) (size 0.3 1.5)
+      (layers F.Cu F.Paste F.Mask)
+    )
+    (pad 7 smd oval (at -0.75 4.75) (size 0.3 1.5)
+      (layers F.Cu F.Paste F.Mask)
+    )
+    (pad 8 smd oval (at -0.25 4.75) (size 0.3 1.5)
+      (layers F.Cu F.Paste F.Mask)
+    )
+    (pad 65 smd rect (at 0 0 90) (size 7 7)
+      (layers F.Cu F.Paste F.Mask)
+    )
+  )
+  (gr_line (start 199.39 158.75) (end 199.39 137.16) (angle 90) (layer Edge.Cuts) (width 0.1))
+  (gr_line (start 224.79 158.75) (end 199.39 158.75) (angle 90) (layer Edge.Cuts) (width 0.1))
+  (gr_line (start 224.79 137.16) (end 224.79 158.75) (angle 90) (layer Edge.Cuts) (width 0.1))
+  (gr_line (start 199.39 137.16) (end 224.79 137.16) (angle 90) (layer Edge.Cuts) (width 0.1))
 )
