File: src/CC3200.sch (KiCad schematic (older format))
At the start: 0 parts

Commit message: Footprint and Symbol updated
Parts:
- added U1: CC3200, ~, symbol CC3200
Changed lines of the file:
@@
 LIBS:contrib
 LIBS:valves
+LIBS:CC3200
 LIBS:CC3200-cache
 EELAYER 27 0
@@
 Sheet 1 1
 Title "CC3200 breakout board"
-Date "14 nov 2014"
+Date "16 nov 2014"
 Rev "A"
 Comp "Turégano"
@@
 Comment4 ""
 $EndDescr
+$Comp
+L CC3200 U1
+U 1 1 54695D9F
+P 5950 4150
+F 0 "U1" H 5950 4200 50  0000 C CNN
+F 1 "CC3200" H 5950 4300 50  0000 C CNN
+F 2 "~" H 5950 2350 60  0000 C CNN
+F 3 "~" H 5950 2350 60  0000 C CNN
+	1    5950 4150
+	1    0    0    -1
+$EndComp
 $EndSCHEMATC
